Commit message: Add files via upload

File: diff_robot/urdf/diff_robot_1cam.xacro (robot description, xacro)
@@ -53,6 +53,4 @@
   <!-- BASE-FOOTPRINT -->
   <!-- base_footprint is a fictitious link(frame) that is on the ground right below base_link origin -->
-  <link name="dummy0">
-   </link>
   <link name="base_footprint">
     <inertial>
@@ -70,17 +68,11 @@
     </visual>
   </link>
-  <joint name="dummy_joint0" type="fixed">
-     <parent link="dummy0"/>
-     <child link="base_footprint"/>
-  </joint>
   <gazebo reference="base_footprint">
     <turnGravityOff>false</turnGravityOff>
   </gazebo>
-  <link name="dummy">
-   </link>
   <joint name="base_footprint_joint" type="fixed">
     <origin xyz="0 0 ${wheel_radius - base_z_origin_to_wheel_origin}" rpy="0 0 0" />
     <parent link="base_footprint"/>
-    <child link="dummy" />
+    <child link="base_link" />
   </joint>
   <!-- BASE-LINK -->
@@ -107,8 +99,4 @@
     </collision>
   </link>
-  <joint name="dummy_joint" type="fixed">
-     <parent link="dummy"/>
-     <child link="base_link"/>
-  </joint>
   <gazebo reference="base_link">
     <material>Gazebo/White</material>
@@ -200,5 +188,5 @@
     <sensor type="ray" name="head_hokuyo_sensor">
       <pose>${hokuyo_size/2} 0 0 0 0 0</pose>
-      <visualize>$(arg viv)</visualize>
+      <visualize>true</visualize>
       <update_rate>40</update_rate>
       <ray>
@@ -207,6 +195,6 @@
             <samples>720</samples>
             <resolution>1</resolution>
-            <min_angle>-6.28</min_angle>
-            <max_angle>6.28</max_angle>
+            <min_angle>-1.570796</min_angle>
+            <max_angle>1.570796</max_angle>
           </horizontal>
         </scan>
@@ -257,4 +245,67 @@
     </sensor>
   </gazebo>
+<joint name="camera_joint" type="fixed">
+    <origin xyz="${base_radius - hokuyo_size/2} 0 ${base_height+hokuyo_size/4+0.1}" rpy="0 0.25 0" />
+    <parent link="base_link"/>
+    <child link="camera_link"/>
+  </joint>
+  <!-- Camera -->
+  <link name="camera_link">
+    <collision>
+      <origin xyz="0 0 0" rpy="0 0 0"/>
+      <geometry>
+    <box size="${camera_link} ${camera_link} ${camera_link}"/>
+      </geometry>
+    </collision>
+    <visual>
+      <origin xyz="0 0 0" rpy="0 0 0"/>
+      <geometry>
+    <box size="${camera_link} ${camera_link} ${camera_link}"/>
+      </geometry>
+      <material name="red"/>
+    </visual>
+    <inertial>
+      <mass value="1e-5" />
+      <origin xyz="0 0 0" rpy="0 0 -1"/>
+      <inertia ixx="1e-6" ixy="0" ixz="0" iyy="1e-6" iyz="0" izz="1e-6" />
+    </inertial>
+  </link>
+   <!-- camera -->
+  <gazebo reference="camera_link">
+      <sensor type="depth" name="camera">
+        <always_on>true</always_on>
+        <update_rate>20.0</update_rate>
+        <camera>
+          <horizontal_fov>${60.0*M_PI/180.0}</horizontal_fov>
+          <image>
+            <format>B8G8R8</format>
+            <width>640</width>
+            <height>480</height>
+          </image>
+          <clip>
+            <near>0.05</near>
+            <far>8.0</far>
+          </clip>
+        </camera>
+        <plugin name="kinect_camera_controller" filename="libgazebo_ros_openni_kinect.so">
+          <cameraName>camera</cameraName>
+          <alwaysOn>true</alwaysOn>
+          <updateRate>10</updateRate>
+          <imageTopicName>rgb/image_raw</imageTopicName>
+          <depthImageTopicName>depth/image_raw</depthImageTopicName>
+          <pointCloudTopicName>depth/points</pointCloudTopicName>
+          <cameraInfoTopicName>rgb/camera_info</cameraInfoTopicName>
+          <depthImageCameraInfoTopicName>depth/camera_info</depthImageCameraInfoTopicName>
+          <frameName>camera_link_optical</frameName>
+          <baseline>0.1</baseline>
+          <distortion_k1>0.0</distortion_k1>
+          <distortion_k2>0.0</distortion_k2>
+          <distortion_k3>0.0</distortion_k3>
+          <distortion_t1>0.0</distortion_t1>
+          <distortion_t2>0.0</distortion_t2>
+          <pointCloudCutoff>0.4</pointCloudCutoff>
+        </plugin>
+      </sensor>
+    </gazebo>
   <!-- Differential drive controller  -->
   <gazebo>

File: diff_robot/urdf/diff_robot_2cam.urdf (robot description, URDF)
Before this commit: robot differential_wheeled_robot, 8 links, 7 joints
Links:
- added link camera1_link, mass 1e-5; collision box size=0.05 0.05 0.05; visual box size=0.05 0.05 0.05
- added link camera2_link, mass 1e-5; collision box size=0.05 0.05 0.05; visual box size=0.05 0.05 0.05
- added link hokuyo_link; visual box size=0.05 0.05 0.05
- added link imu_link; visual box size=0.05 0.05 0.05
Joints:
- added joint camera1_joint: type fixed, parent base_link, child camera1_link, origin xyz=0.125 0.06 0.1325 rpy=0 0 0
- added joint camera2_joint: type fixed, parent base_link, child camera2_link, origin xyz=0.125 -0.06 0.1325 rpy=0 0 0
- added joint hokuyo_joint: type fixed, parent base_link, child hokuyo_link, origin xyz=0.125 0 0.0325 rpy=0 0 0
- added joint imu_joint: type fixed, parent base_link, child imu_link, origin xyz=0.075 0.1 0.0325 rpy=0 0 0

File: diff_robot/urdf/diff_robot_2cam.xacro (robot description, xacro)
@@ -1,4 +1,4 @@
 <?xml version="1.0"?>
-<robot name="differential_wheeled_robot" xmlns:xacro="http://ros.org/wiki/xacro">
+<robot name="cam_robot" xmlns:xacro="http://ros.org/wiki/xacro">
   <xacro:include filename="$(find diff_robot)/urdf/wheel.urdf.xacro" />
   <xacro:property name="camera_link" value="0.05" /> <!-- Size of square 'camera' box -->
@@ -200,5 +200,5 @@
     <sensor type="ray" name="head_hokuyo_sensor">
       <pose>${hokuyo_size/2} 0 0 0 0 0</pose>
-      <visualize>$(arg viv)</visualize>
+      <visualize>true</visualize>
       <update_rate>40</update_rate>
       <ray>
@@ -207,6 +207,6 @@
             <samples>720</samples>
             <resolution>1</resolution>
-            <min_angle>-6.28</min_angle>
-            <max_angle>6.28</max_angle>
+            <min_angle>-1.570796</min_angle>
+            <max_angle>1.570796</max_angle>
           </horizontal>
         </scan>
@@ -257,4 +257,130 @@
     </sensor>
   </gazebo>
+<joint name="camera1_joint" type="fixed">
+    <origin xyz="${base_radius - hokuyo_size/2} 0.06 ${base_height+hokuyo_size/4+0.1}" rpy="0 0 0" />
+    <parent link="base_link"/>
+    <child link="camera1_link"/>
+  </joint>
+  <!-- Camera -->
+  <link name="camera1_link">
+    <collision>
+      <origin xyz="0 0 0" rpy="0 0 0"/>
+      <geometry>
+    <box size="${camera_link} ${camera_link} ${camera_link}"/>
+      </geometry>
+    </collision>
+    <visual>
+      <origin xyz="0 0 0" rpy="0 0 0"/>
+      <geometry>
+    <box size="${camera_link} ${camera_link} ${camera_link}"/>
+      </geometry>
+      <material name="red"/>
+    </visual>
+    <inertial>
+      <mass value="1e-5" />
+      <origin xyz="${base_radius - hokuyo_size/2} 0.06 ${base_height+hokuyo_size/4+0.1}" rpy="0 0 0"/>
+      <inertia ixx="1e-6" ixy="0" ixz="0" iyy="1e-6" iyz="0" izz="1e-6" />
+    </inertial>
+  </link>
+   <!-- camera -->
+  <gazebo reference="camera1_link">
+      <sensor type="depth" name="camera1">
+        <always_on>true</always_on>
+        <update_rate>20.0</update_rate>
+        <camera>
+          <horizontal_fov>${60.0*M_PI/180.0}</horizontal_fov>
+          <image>
+            <format>B8G8R8</format>
+            <width>640</width>
+            <height>480</height>
+          </image>
+          <clip>
+            <near>0.05</near>
+            <far>8.0</far>
+          </clip>
+        </camera>
+        <plugin name="kinect_camera_controller" filename="libgazebo_ros_openni_kinect.so">
+          <cameraName>camera</cameraName>
+          <alwaysOn>true</alwaysOn>
+          <updateRate>10</updateRate>
+          <imageTopicName>rgb/image_raw1</imageTopicName>
+          <depthImageTopicName>depth/image_raw1</depthImageTopicName>
+          <pointCloudTopicName>depth/points1</pointCloudTopicName>
+          <cameraInfoTopicName>rgb/camera_info1</cameraInfoTopicName>
+          <depthImageCameraInfoTopicName>depth/camera_info1</depthImageCameraInfoTopicName>
+          <frameName>camera_link_optical</frameName>
+          <baseline>0.1</baseline>
+          <distortion_k1>0.0</distortion_k1>
+          <distortion_k2>0.0</distortion_k2>
+          <distortion_k3>0.0</distortion_k3>
+          <distortion_t1>0.0</distortion_t1>
+          <distortion_t2>0.0</distortion_t2>
+          <pointCloudCutoff>0.4</pointCloudCutoff>
+        </plugin>
+      </sensor>
+    </gazebo>
+  <joint name="camera2_joint" type="fixed">
+    <origin xyz="${base_radius - hokuyo_size/2} -0.06 ${base_height+hokuyo_size/4+0.1}" rpy="0 0 0" />
+    <parent link="base_link"/>
+    <child link="camera2_link"/>
+  </joint>
+  <!-- Camera -->
+  <link name="camera2_link">
+    <collision>
+      <origin xyz="0 0 0" rpy="0 0 0"/>
+      <geometry>
+    <box size="${camera_link} ${camera_link} ${camera_link}"/>
+      </geometry>
+    </collision>
+    <visual>
+      <origin xyz="0 0 0" rpy="0 0 0"/>
+      <geometry>
+    <box size="${camera_link} ${camera_link} ${camera_link}"/>
+      </geometry>
+      <material name="red"/>
+    </visual>
+    <inertial>
+      <mass value="1e-5" />
+      <origin xyz="${base_radius - hokuyo_size/2} -0.06 ${base_height+hokuyo_size/4+0.1}" rpy="0 0 0"/>
+      <inertia ixx="1e-6" ixy="0" ixz="0" iyy="1e-6" iyz="0" izz="1e-6" />
+    </inertial>
+  </link>
+   <!-- camera -->
+  <gazebo reference="camera2_link">
+      <sensor type="depth" name="camera2">
+        <always_on>true</always_on>
+        <update_rate>20.0</update_rate>
+        <camera>
+          <horizontal_fov>${60.0*M_PI/180.0}</horizontal_fov>
+          <image>
+            <format>B8G8R8</format>
+            <width>640</width>
+            <height>480</height>
+          </image>
+          <clip>
+            <near>0.05</near>
+            <far>8.0</far>
+          </clip>
+        </camera>
+        <plugin name="kinect_camera_controller" filename="libgazebo_ros_openni_kinect.so">
+          <cameraName>camera</cameraName>
+          <alwaysOn>true</alwaysOn>
+          <updateRate>10</updateRate>
+          <imageTopicName>rgb/image_raw2</imageTopicName>
+          <depthImageTopicName>depth/image_raw2</depthImageTopicName>
+          <pointCloudTopicName>depth/points2</pointCloudTopicName>
+          <cameraInfoTopicName>rgb/camera_info2</cameraInfoTopicName>
+          <depthImageCameraInfoTopicName>depth/camera_info2</depthImageCameraInfoTopicName>
+          <frameName>camera_link_optical</frameName>
+          <baseline>0.1</baseline>
+          <distortion_k1>0.0</distortion_k1>
+          <distortion_k2>0.0</distortion_k2>
+          <distortion_k3>0.0</distortion_k3>
+          <distortion_t1>0.0</distortion_t1>
+          <distortion_t2>0.0</distortion_t2>
+          <pointCloudCutoff>0.4</pointCloudCutoff>
+        </plugin>
+      </sensor>
+    </gazebo>
   <!-- Differential drive controller  -->
   <gazebo>

File: diff_robot/urdf/diff_wheeled_robot_with_laser.urdf (robot description, URDF)
Before this commit: robot differential_wheeled_robot, 8 links, 7 joints
Links:
- added link camera_link, mass 1e-5; collision box size=0.05 0.05 0.05; visual box size=0.05 0.05 0.05
- added link hokuyo_link; visual box size=0.05 0.05 0.05
- added link imu_link; visual box size=0.05 0.05 0.05
Joints:
- added joint camera_joint: type fixed, parent base_link, child camera_link, origin xyz=0.125 0 0.1325 rpy=0 0 0
- added joint hokuyo_joint: type fixed, parent base_link, child hokuyo_link, origin xyz=0.125 0 0.0325 rpy=0 0 0
- added joint imu_joint: type fixed, parent base_link, child imu_link, origin xyz=0.075 0.1 0.0325 rpy=0 0 0
